Commit message: initial fixes for IAwake robot

File: op3_description/urdf/robotis_op3.gazebo.xacro (robot description, xacro)
@@ -117,5 +117,4 @@
     <mu1>0.2</mu1>
     <mu2>0.2</mu2>
-    <material>Gazebo/White</material>
     <selfCollide>false</selfCollide>
   </gazebo>
@@ -123,5 +122,9 @@
     <mu1>0.2</mu1>
     <mu2>0.2</mu2>
-    <material>Gazebo/White</material>
+    <selfCollide>false</selfCollide>
+  </gazebo>
+  <gazebo reference="l_sho_yaw_link">
+    <mu1>0.2</mu1>
+    <mu2>0.2</mu2>
     <selfCollide>false</selfCollide>
   </gazebo>
@@ -129,5 +132,4 @@
     <mu1>0.2</mu1>
     <mu2>0.2</mu2>
-    <material>Gazebo/White</material>
     <selfCollide>false</selfCollide>
   </gazebo>

File: op3_description/urdf/robotis_op3.inertia.xacro (robot description, xacro)
@@ -146,4 +146,12 @@
              izz="0.00023474" />
   </xacro:macro>
+  <!-- left shoulder yaw joint -->
+  <xacro:macro name="insert_inertia_l_sho_yaw_link">
+    <origin xyz="-0.01844 0.04514 0.00028" />
+    <mass value="0.17758"/>
+    <inertia ixx="0.00022804" ixy="-0.00000001" ixz="0.00000003"
+             iyy="0.00003042" iyz="0.00000059"
+             izz="0.00023474" />
+  </xacro:macro>
   <!-- left elbow joint -->
   <xacro:macro name="insert_inertia_l_el_link">

File: op3_description/urdf/robotis_op3.structure.lleg.xacro (robot description, xacro)
@@ -82,5 +82,5 @@
   </joint>
   <xacro:insert_transmission name="l_knee" />
-  <!-- left hip pitch link -->
+  <!-- left knee link -->
   <link name="l_knee_link">
     <visual>
@@ -104,5 +104,5 @@
   </joint>
   <xacro:insert_transmission name="l_ank_pitch" />
-  <!-- left hip pitch link -->
+  <!-- left ankle pitch link -->
   <link name="l_ank_pitch_link">
     <visual>
@@ -117,4 +117,5 @@
   </link>
   <!-- left ankle roll link -->
+  <!--
   <joint name="l_ank_roll" type="revolute">
     <parent link="l_ank_pitch_link"/>
@@ -126,5 +127,7 @@
   </joint>
   <xacro:insert_transmission name="l_ank_roll" />
+  -->
   <!-- left hip roll link -->
+  <!--
   <link name="l_ank_roll_link">
     <visual>
@@ -138,4 +141,5 @@
     </inertial>
   </link>
+  -->
   </xacro:macro>
 </robot>

File: op3_description/urdf/robotis_op3.visuals.xacro (robot description, xacro)
@@ -144,5 +144,5 @@
     </material>
   </xacro:macro>
-  <!-- right shoulder pitch joint -->
+  <!-- right shoulder roll joint -->
   <xacro:macro name="insert_mesh_r_sho_roll_link">
     <origin xyz="0 0 0" rpy="0 0 0" />
@@ -168,31 +168,41 @@
     <origin xyz="0 0 0" rpy="0 0 0" />
     <geometry>
-      <mesh filename="package://op3_description/meshes/la1.stl"  scale="0.001 0.001 0.001"/>
-    </geometry>
-    <material name="Grey">
-      <color rgba="0.60 0.60 0.60 1.0"/>
-    </material>
-  </xacro:macro>
-  <!-- left shoulder pitch joint -->
+      <mesh filename="package://op3_description/meshes/l_shoulder_visual.STL"/>
+    </geometry>
+    <material name="Grey">
+      <color rgba="0.60 0.60 0.60 1.0"/>
+    </material>
+  </xacro:macro>
+  <!-- left shoulder roll joint -->
   <xacro:macro name="insert_mesh_l_sho_roll_link">
     <origin xyz="0 0 0" rpy="0 0 0" />
     <geometry>
-      <mesh filename="package://op3_description/meshes/la2.stl"  scale="0.001 0.001 0.001"/>
-    </geometry>
-    <material name="Grey">
-      <color rgba="0.60 0.60 0.60 1.0"/>
-    </material>
-  </xacro:macro>
-  <!-- left elbow joint -->
+      <mesh filename="package://op3_description/meshes/l_upper_arm_visual.STL"/>
+    </geometry>
+    <material name="Grey">
+      <color rgba="0.60 0.60 0.60 1.0"/>
+    </material>
+  </xacro:macro>
+  <!-- left shoulder yaw joint -->
+  <xacro:macro name="insert_mesh_l_sho_yaw_link">
+    <origin xyz="0 0 0" rpy="0 0 0" />
+    <geometry>
+      <mesh filename="package://op3_description/meshes/l_shoulder_motor_visual.STL"/>
+    </geometry>
+    <material name="Grey">
+      <color rgba="0.60 0.60 0.60 1.0"/>
+    </material>
+  </xacro:macro>
+    <!-- left elbow joint -->
   <xacro:macro name="insert_mesh_l_el_link">
     <origin xyz="0 0 0" rpy="0 0 0" />
     <geometry>
-      <mesh filename="package://op3_description/meshes/la3.stl"  scale="0.001 0.001 0.001"/>
-    </geometry>
-    <material name="Grey">
-      <color rgba="0.60 0.60 0.60 1.0"/>
-    </material>
-  </xacro:macro>
-  <!-- head yaw joint -->
+      <mesh filename="package://op3_description/meshes/l_forearm_visual.STL"/>
+    </geometry>
+    <material name="Grey">
+      <color rgba="0.60 0.60 0.60 1.0"/>
+    </material>
+  </xacro:macro>
+  <!-- head pan joint -->
   <xacro:macro name="insert_mesh_head_pan_link">
     <origin xyz="0 0 0" rpy="0 0 0" />
@@ -204,5 +214,5 @@
     </material>
   </xacro:macro>
-  <!-- head yaw joint -->
+  <!-- head tilt joint -->
   <xacro:macro name="insert_mesh_head_tilt_link">
     <origin xyz="0 0 0" rpy="0 0 0" />
