Commit message: fixes for simulator, head model

File: op3_description/urdf/OP3_IAwake.urdf (robot description, URDF)
Before this commit: robot robotis_op3, 24 links, 23 joints
Links:
- added link head, mass 0.5; visual mesh filename=package://op3_description/meshes/head_01-copy-tenth-scale02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 scale=0.0009 0.0009 0.0009
Joints:
- added joint head_pan: type revolute, parent pelvis, child head, origin xyz=0.0 -0.1 0.245 rpy=0 0 0, axis 0 0 1, limit lower=-0.497418836818 upper=0.523598775598 effort=3.1 velocity=7.0

Commit message: updates after kinematics changes

File: op3_description/urdf/OP3_IAwake.urdf (robot description, URDF)
Before this commit: robot robotis_op3, 25 links, 24 joints
Links:
- link head: geometry visual mesh filename=package://op3_description/meshes/head_01-copy-tenth-scale02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 scale=0.0007 0.0007 0.0007
Joints:
- joint head_pan: origin xyz=0.0 -0.1 0.245 rpy=0 0 0 -> xyz=0.0 -0.1 0.345 rpy=0 0 0
- joint l_hip_yaw: origin xyz=0.0439986111539757 0 0.005 rpy=0 0 0 -> xyz=0.0439986111539757 0 0.005 rpy=0 -0.523598775596 0
- joint l_sho_yaw: origin xyz=0 0.03625 0.0185000000000001 rpy=0 0 0 -> xyz=0 0.03625 0.0185000000000001 rpy=0 1.5707963267949 0
- joint r_hip_yaw: origin xyz=-0.0439986111539757 0 0.005 rpy=0 0 0 -> xyz=-0.0439986111539757 0 0.005 rpy=0 0.523598775596 0
- joint r_sho_yaw: origin xyz=0 0.03625 0.0185000000000002 rpy=0 0 0 -> xyz=0 0.03625 0.0185000000000002 rpy=0 -1.5707963267949 0
